File: sop28-to-dip-24-rom-adapter.kicad_pcb (KiCad board)
At the start: 2 copper layers, 20.3 x 33 mm, 3 parts, among them U2 ROM_24

Commit message: Revision 3.
Parts:
- added R2: 10K, Resistor_THT:R_Axial_DIN0207_L6.3mm_D2.5mm_P10.16mm_Horizontal, F.Cu at (129.5, 83.8)
- renumbered 10K to R1, 28C64 to U1
Connections:
- U1 pad 1: unconnected-(U1-RDY/~{BUSY}-Pad1) -> Net-(U1-RDY/~{BUSY})
Routing:
- net GND: track 27.1 -> 37.4 mm, vias 0 -> 1
- net Net-(U1-RDY/~{BUSY}): track 0.00 -> 3.23 mm
- net VCC: track 8.28 -> 8.85 mm
- net Net-(U1-~{WE}): vias 0 -> 1
Other:
- board text added: "SOP-28"
- board text removed: "SOIC-28"
Changed lines of the file:
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@@
   (paper "A4")
   (title_block
-    (title "SOP-28 to DIP-24 ROM adapter.")
-    (date "2024-03-24")
-    (rev "2")
+    (title "SOP-28 to DIP-24 ROM adaptor.")
+    (date "2024-04-14")
+    (rev "3")
     (company "Thierry Tremblay")
   )
@@
   (net 23 "/A8")
   (net 24 "VCC")
-  (net 25 "unconnected-(U1-RDY{slash}~{BUSY}-Pad1)")
+  (net 25 "Net-(U1-RDY{slash}~{BUSY})")
   (net 26 "Net-(U1-~{CS})")
   (footprint "Resistor_THT:R_Axial_DIN0207_L6.3mm_D2.5mm_P10.16mm_Horizontal" (layer "F.Cu")
@@
     (property "ki_keywords" "R res resistor")
     (attr through_hole)
-    (fp_text reference "10K" (at 5.08 0) (layer "F.SilkS")
+    (fp_text reference "R1" (at 5.08 0) (layer "F.SilkS")
         (effects (font (size 1 1) (thickness 0.15)))
     )
@@
     (property "ki_keywords" "Parallel EEPROM 256Kb")
     (attr smd)
-    (fp_text reference "28C64" (at 0.155 11.425) (layer "F.SilkS")
+    (fp_text reference "U1" (at 0.155 11.425) (layer "F.SilkS")
         (effects (font (size 1 1) (thickness 0.15)))
     )
@@
       (stroke (width 0.1) (type solid)) (layer "F.Fab"))
     (pad "1" smd roundrect (at -4.8 -8.255) (size 1.8 0.6) (layers "F.Cu" "F.Paste" "F.Mask") (roundrect_rratio 0.25)
-      (net 25 "unconnected-(U1-RDY{slash}~{BUSY}-Pad1)") (pinfunction "RDY/~{BUSY}") (pintype "output"))
+      (net 25 "Net-(U1-RDY{slash}~{BUSY})") (pinfunction "RDY/~{BUSY}") (pintype "output"))
     (pad "2" smd roundrect (at -4.8 -6.985) (size 1.8 0.6) (layers "F.Cu" "F.Paste" "F.Mask") (roundrect_rratio 0.25)
       (net 2 "/A12") (pinfunction "A12") (pintype "input"))
@@
     )
   )
+  (footprint "Resistor_THT:R_Axial_DIN0207_L6.3mm_D2.5mm_P10.16mm_Horizontal" (layer "F.Cu")
+    (at 129.54 83.82)
+    (descr "Resistor, Axial_DIN0207 series, Axial, Horizontal, pin pitch=10.16mm, 0.25W = 1/4W, length*diameter=6.3*2.5mm^2, http://cdn-reichelt.de/documents/datenblatt/B400/1_4W%23YAG.pdf")
+    (tags "Resistor Axial_DIN0207 series Axial Horizontal pin pitch 10.16mm 0.25W = 1/4W length 6.3mm diameter 2.5mm")
+    (property "Sheetfile" "sop28-to-dip-24-rom-adapter.kicad_sch")
+    (property "Sheetname" "")
+    (property "ki_description" "Resistor")
+    (property "ki_keywords" "R res resistor")
+    (attr through_hole)
+    (fp_text reference "R2" (at 5.08 -2.37) (layer "F.SilkS")
+        (effects (font (size 1 1) (thickness 0.15)))
+    )
+    (fp_text value "10K" (at 5.08 2.37) (layer "F.Fab")
+        (effects (font (size 1 1) (thickness 0.15)))
+    )
+    (fp_text user "${REFERENCE}" (at 5.08 0) (layer "F.Fab")
+        (effects (font (size 1 1) (thickness 0.15)))
+    )
+    (fp_line (start 1.04 0) (end 1.81 0)
+      (stroke (width 0.12) (type solid)) (layer "F.SilkS"))
+    (fp_line (start 1.81 -1.37) (end 1.81 1.37)
+      (stroke (width 0.12) (type solid)) (layer "F.SilkS"))
+    (fp_line (start 1.81 1.37) (end 8.35 1.37)
+      (stroke (width 0.12) (type solid)) (layer "F.SilkS"))
+    (fp_line (start 8.35 -1.37) (end 1.81 -1.37)
+      (stroke (width 0.12) (type solid)) (layer "F.SilkS"))
+    (fp_line (start 8.35 1.37) (end 8.35 -1.37)
+      (stroke (width 0.12) (type solid)) (layer "F.SilkS"))
+    (fp_line (start 9.12 0) (end 8.35 0)
+      (stroke (width 0.12) (type solid)) (layer "F.SilkS"))
+    (fp_line (start -1.05 -1.5) (end -1.05 1.5)
+      (stroke (width 0.05) (type solid)) (layer "F.CrtYd"))
+    (fp_line (start -1.05 1.5) (end 11.21 1.5)
+      (stroke (width 0.05) (type solid)) (layer "F.CrtYd"))
+    (fp_line (start 11.21 -1.5) (end -1.05 -1.5)
+      (stroke (width 0.05) (type solid)) (layer "F.CrtYd"))
+    (fp_line (start 11.21 1.5) (end 11.21 -1.5)
+      (stroke (width 0.05) (type solid)) (layer "F.CrtYd"))
+    (fp_line (start 0 0) (end 1.93 0)
+      (stroke (width 0.1) (type solid)) (layer "F.Fab"))
+    (fp_line (start 1.93 -1.25) (end 1.93 1.25)
+      (stroke (width 0.1) (type solid)) (layer "F.Fab"))
+    (fp_line (start 1.93 1.25) (end 8.23 1.25)
+      (stroke (width 0.1) (type solid)) (layer "F.Fab"))
+    (fp_line (start 8.23 -1.25) (end 1.93 -1.25)
+      (stroke (width 0.1) (type solid)) (layer "F.Fab"))
+    (fp_line (start 8.23 1.25) (end 8.23 -1.25)
+      (stroke (width 0.1) (type solid)) (layer "F.Fab"))
+    (fp_line (start 10.16 0) (end 8.23 0)
+      (stroke (width 0.1) (type solid)) (layer "F.Fab"))
+    (pad "1" thru_hole circle (at 0 0) (size 1.6 1.6) (drill 0.8) (layers "*.Cu" "*.Mask")
+      (net 25 "Net-(U1-RDY{slash}~{BUSY})") (pintype "passive"))
+    (pad "2" thru_hole oval (at 10.16 0) (size 1.6 1.6) (drill 0.8) (layers "*.Cu" "*.Mask")
+      (net 1 "GND") (pintype "passive"))
+    (model "${KICAD6_3DMODEL_DIR}/Resistor_THT.3dshapes/R_Axial_DIN0207_L6.3mm_D2.5mm_P10.16mm_Horizontal.wrl"
+      (offset (xyz 0 0 0))
+      (scale (xyz 1 1 1))
+      (rotate (xyz 0 0 0))
+    )
+  )
   (footprint "Library:DIP-24_W15.24mm-Notch" (layer "F.Cu")
     (at 126.84 81.28)
@@
     (effects (font (size 1 1) (thickness 0.15)) (justify left bottom mirror))
   )
-  (gr_text "SOIC-28" (at 134.62 109.22) (layer "F.SilkS")
+  (gr_text "SOP-28" (at 134.62 109.22) (layer "F.SilkS")
     (effects (font (size 1 1) (thickness 0.15)))
   )
-  (segment (start 134.62 93.285001) (end 138.365001 89.54) (width 0.25) (layer "F.Cu") (net 1))
+  (segment (start 136.435 91.470002) (end 135.542501 92.362501) (width 0.25) (layer "F.Cu") (net 1))
+  (segment (start 136.435 87.085) (end 136.435 91.470002) (width 0.25) (layer "F.Cu") (net 1))
+  (segment (start 135.542501 92.362501) (end 138.365001 89.54) (width 0.25) (layer "F.Cu") (net 1))
   (segment (start 126.84 109.22) (end 129.665 106.395) (width 0.25) (layer "F.Cu") (net 1))
   (segment (start 134.62 101.6) (end 134.62 93.285001) (width 0.25) (layer "F.Cu") (net 1))
+  (segment (start 134.62 93.285001) (end 135.542501 92.362501) (width 0.25) (layer "F.Cu") (net 1))
   (segment (start 129.665 106.395) (end 129.665 103.51) (width 0.25) (layer "F.Cu") (net 1))
   (segment (start 138.365001 89.54) (end 139.265 89.54) (width 0.25) (layer "F.Cu") (net 1))
   (segment (start 129.665 103.51) (end 132.71 103.51) (width 0.25) (layer "F.Cu") (net 1))
+  (segment (start 137.16 86.36) (end 136.435 87.085) (width 0.25) (layer "F.Cu") (net 1))
   (segment (start 132.71 103.51) (end 134.62 101.6) (width 0.25) (layer "F.Cu") (net 1))
+  (via (at 137.16 86.36) (size 0.8) (drill 0.4) (layers "F.Cu" "B.Cu") (net 1))
+  (segment (start 139.7 83.82) (end 137.16 86.36) (width 0.25) (layer "B.Cu") (net 1))
   (segment (start 133.99 88.27) (end 129.665 88.27) (width 0.25) (layer "F.Cu") (net 2))
   (segment (start 134.62 88.9) (end 133.99 88.27) (width 0.25) (layer "F.Cu") (net 2))
@@
   (segment (start 139.265 98.43) (end 141.45 98.43) (width 0.25) (layer "F.Cu") (net 18))
   (segment (start 141.45 98.43) (end 142.08 99.06) (width 0.25) (layer "F.Cu") (net 18))
-  (segment (start 136.53 88.27) (end 139.265 88.27) (width 0.25) (layer "F.Cu") (net 19))
-  (segment (start 129.54 81.28) (end 136.53 88.27) (width 0.25) (layer "F.Cu") (net 19))
+  (segment (start 139.1705 88.1755) (end 139.265 88.27) (width 0.25) (layer "F.Cu") (net 19))
+  (segment (start 137.16 88.1755) (end 139.1705 88.1755) (width 0.25) (layer "F.Cu") (net 19))
+  (via (at 137.16 88.1755) (size 0.8) (drill 0.4) (layers "F.Cu" "B.Cu") (net 19))
+  (segment (start 136.4355 88.1755) (end 137.16 88.1755) (width 0.25) (layer "B.Cu") (net 19))
+  (segment (start 129.54 81.28) (end 136.4355 88.1755) (width 0.25) (layer "B.Cu") (net 19))
   (segment (start 139.265 95.89) (end 140.17 95.89) (width 0.25) (layer "F.Cu") (net 20))
   (segment (start 140.17 95.89) (end 142.08 93.98) (width 0.25) (layer "F.Cu") (net 20))
@@
   (segment (start 140.49 90.65) (end 140.33 90.81) (width 0.25) (layer "F.Cu") (net 23))
   (segment (start 140.33 90.81) (end 139.265 90.81) (width 0.25) (layer "F.Cu") (net 23))
-  (segment (start 139.265 87) (end 139.7 86.565) (width 0.25) (layer "F.Cu") (net 24))
+  (segment (start 138.575 86.31) (end 139.265 87) (width 0.25) (layer "F.Cu") (net 24))
+  (segment (start 138.575 82.405) (end 138.575 86.31) (width 0.25) (layer "F.Cu") (net 24))
+  (segment (start 139.7 81.28) (end 138.575 82.405) (width 0.25) (layer "F.Cu") (net 24))
   (segment (start 142.08 81.28) (end 139.7 81.28) (width 0.25) (layer "F.Cu") (net 24))
-  (segment (start 139.7 86.565) (end 139.7 81.28) (width 0.25) (layer "F.Cu") (net 24))
+  (segment (start 129.54 86.875) (end 129.665 87) (width 0.25) (layer "F.Cu") (net 25))
+  (segment (start 129.54 83.82) (end 129.54 86.875) (width 0.25) (layer "F.Cu") (net 25))
   (segment (start 142.08 91.44) (end 142.08 92.110908) (width 0.25) (layer "F.Cu") (net 26))
   (segment (start 138.365001 97.16) (end 138.04 96.834999) (width 0.25) (layer "F.Cu") (net 26))
