File: sop28-to-dip-24-rom-adapter.kicad_pcb (KiCad board)
At the start: 2 copper layers, 20.3 x 33 mm, 3 parts, among them U2 ROM_24

Commit message: Revision 2B.
Parts:
- 4.7K: renamed from 10K; value 10K -> 4.7K
- moved 4.7K 1.27 mm to (139.7, 82.5)
Routing:
- net VCC: track 8.28 -> 7.54 mm
- net Net-(U1-~{WE}): track 12.6 -> 12.1 mm
Other:
- board size 20.3 x 33 mm -> 17.8 x 30.5 mm
- board text added: "Revision 2B"
- board text removed: "Revision 2"
Changed lines of the file:
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@@
     (title "SOP-28 to DIP-24 ROM adapter.")
     (date "2024-03-24")
-    (rev "2")
+    (rev "2B")
     (company "Thierry Tremblay")
   )
@@
   (net 26 "Net-(U1-~{CS})")
   (footprint "Resistor_THT:R_Axial_DIN0207_L6.3mm_D2.5mm_P10.16mm_Horizontal" (layer "F.Cu")
-    (at 139.7 81.28 180)
+    (at 139.7 82.55 180)
     (descr "Resistor, Axial_DIN0207 series, Axial, Horizontal, pin pitch=10.16mm, 0.25W = 1/4W, length*diameter=6.3*2.5mm^2, http://cdn-reichelt.de/documents/datenblatt/B400/1_4W%23YAG.pdf")
     (tags "Resistor Axial_DIN0207 series Axial Horizontal pin pitch 10.16mm 0.25W = 1/4W length 6.3mm diameter 2.5mm")
@@
     (property "ki_keywords" "R res resistor")
     (attr through_hole)
-    (fp_text reference "10K" (at 5.08 0) (layer "F.SilkS")
-        (effects (font (size 1 1) (thickness 0.15)))
-    )
-    (fp_text value "10K" (at 5.08 2.37) (layer "F.Fab")
+    (fp_text reference "4.7K" (at 5.08 0) (layer "F.SilkS")
+        (effects (font (size 1 1) (thickness 0.15)))
+    )
+    (fp_text value "4.7K" (at 5.08 2.37) (layer "F.Fab")
         (effects (font (size 1 1) (thickness 0.15)))
     )
@@
     )
   )
-  (gr_rect (start 124.46 78.74) (end 144.78 111.76)
+  (gr_rect (start 125.73 80.01) (end 143.51 110.49)
     (stroke (width 0.1) (type default)) (fill none) (layer "Edge.Cuts"))
   (gr_text "EEPROM 28C64 to ROM 2364\n" (at 132.08 83.82 90) (layer "B.SilkS")
@@
     (effects (font (size 1 1) (thickness 0.15)) (justify left bottom mirror))
   )
-  (gr_text "Revision 2" (at 137.16 83.82 90) (layer "B.SilkS")
+  (gr_text "Revision 2B" (at 137.16 83.82 90) (layer "B.SilkS")
     (effects (font (size 1 1) (thickness 0.15)) (justify left bottom mirror))
   )
@@
   (segment (start 139.265 98.43) (end 141.45 98.43) (width 0.25) (layer "F.Cu") (net 18))
   (segment (start 141.45 98.43) (end 142.08 99.06) (width 0.25) (layer "F.Cu") (net 18))
-  (segment (start 136.53 88.27) (end 139.265 88.27) (width 0.25) (layer "F.Cu") (net 19))
-  (segment (start 129.54 81.28) (end 136.53 88.27) (width 0.25) (layer "F.Cu") (net 19))
+  (segment (start 139.265 88.27) (end 135.26 88.27) (width 0.25) (layer "F.Cu") (net 19))
+  (segment (start 135.26 88.27) (end 129.54 82.55) (width 0.25) (layer "F.Cu") (net 19))
   (segment (start 139.265 95.89) (end 140.17 95.89) (width 0.25) (layer "F.Cu") (net 20))
   (segment (start 140.17 95.89) (end 142.08 93.98) (width 0.25) (layer "F.Cu") (net 20))
@@
   (segment (start 140.49 90.65) (end 140.33 90.81) (width 0.25) (layer "F.Cu") (net 23))
   (segment (start 140.33 90.81) (end 139.265 90.81) (width 0.25) (layer "F.Cu") (net 23))
+  (segment (start 139.7 82.55) (end 140.97 81.28) (width 0.25) (layer "F.Cu") (net 24))
   (segment (start 139.265 87) (end 139.7 86.565) (width 0.25) (layer "F.Cu") (net 24))
-  (segment (start 142.08 81.28) (end 139.7 81.28) (width 0.25) (layer "F.Cu") (net 24))
-  (segment (start 139.7 86.565) (end 139.7 81.28) (width 0.25) (layer "F.Cu") (net 24))
+  (segment (start 140.97 81.28) (end 142.08 81.28) (width 0.25) (layer "F.Cu") (net 24))
+  (segment (start 139.7 86.565) (end 139.7 82.55) (width 0.25) (layer "F.Cu") (net 24))
   (segment (start 142.08 91.44) (end 142.08 92.110908) (width 0.25) (layer "F.Cu") (net 26))
   (segment (start 138.365001 97.16) (end 138.04 96.834999) (width 0.25) (layer "F.Cu") (net 26))
